File: GPS.kicad_sch (KiCad schematic)
At the start: 3 parts

Commit message: updates to schematics
Parts:
- C201: value (none) -> 0.01uF; footprint (none) -> Capacitor_SMD:C_0603_1608Metric_Pad1.08x0.95mm_HandSolder
- J201: value (none) -> Conn_Coaxial; footprint (none) -> Connector_Coaxial:SMA_Amphenol_901-144_Vertical
- U201: value (none) -> RXM-GPS-RM-T; footprint (none) -> Linx GPS:RXM-GPS-RM-T
Changed lines of the file:
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@@
     (in_bom yes) (on_board yes) (fields_autoplaced)
     (property "Reference" "J201" (id 0) (at 170.4732 63.5 90))
-    (property "Value" "" (id 1) (at 170.4732 66.04 90))
-    (property "Footprint" "" (id 2) (at 170.18 70.485 0)
+    (property "Value" "Conn_Coaxial" (id 1) (at 170.4732 66.04 90))
+    (property "Footprint" "Connector_Coaxial:SMA_Amphenol_901-144_Vertical" (id 2) (at 170.18 70.485 0)
       (effects (font (size 1.27 1.27)) hide)
     )
@@
       (effects (font (size 1.524 1.524)))
     )
-    (property "Value" "" (id 1) (at 135.89 71.12 0)
+    (property "Value" "RXM-GPS-RM-T" (id 1) (at 135.89 71.12 0)
       (effects (font (size 1.524 1.524)))
     )
-    (property "Footprint" "" (id 2) (at 135.89 72.644 0)
+    (property "Footprint" "Linx GPS:RXM-GPS-RM-T" (id 2) (at 135.89 72.644 0)
       (effects (font (size 1.524 1.524)) hide)
     )
@@
       (effects (font (size 1.27 1.27)) hide)
     )
-    (property "Value" "" (id 1) (at 168.275 86.36 0))
+    (property "Value" "GND" (id 1) (at 168.275 86.36 0))
     (property "Footprint" "" (id 2) (at 168.275 91.44 0)
       (effects (font (size 1.27 1.27)) hide)
@@
       (effects (font (size 1.27 1.27)) hide)
     )
-    (property "Value" "" (id 1) (at 105.41 96.52 0))
+    (property "Value" "GND" (id 1) (at 105.41 96.52 0))
     (property "Footprint" "" (id 2) (at 105.41 91.44 0)
       (effects (font (size 1.27 1.27)) hide)
@@
       (effects (font (size 1.27 1.27)) hide)
     )
-    (property "Value" "" (id 1) (at 179.07 70.4849 90)
+    (property "Value" "GND" (id 1) (at 179.07 70.4849 90)
       (effects (font (size 1.27 1.27)) (justify right))
     )
@@
       (effects (font (size 1.27 1.27)) hide)
     )
-    (property "Value" "" (id 1) (at 189.23 101.3717 90)
+    (property "Value" "GND" (id 1) (at 189.23 101.3717 90)
       (effects (font (size 1.27 1.27)) (justify right))
     )
@@
     (in_bom yes) (on_board yes) (fields_autoplaced)
     (property "Reference" "C201" (id 0) (at 173.355 93.98 90))
-    (property "Value" "" (id 1) (at 173.355 96.52 90))
-    (property "Footprint" "" (id 2) (at 177.165 100.6348 0)
+    (property "Value" "0.01uF" (id 1) (at 173.355 96.52 90))
+    (property "Footprint" "Capacitor_SMD:C_0603_1608Metric_Pad1.08x0.95mm_HandSolder" (id 2) (at 177.165 100.6348 0)
       (effects (font (size 1.27 1.27)) hide)
     )
