File: Flight ComputerV1.kicad_sch (KiCad schematic)
At the start: 28 parts, among them J101 ICSP, J102 Screw_Terminal_01x02, J103 Conn_01x08, J104 Conn_01x07, J105 Micro_SD_Card, J106 Conn_02x10_Top_Bottom, SW101 1-1825910-8, U101 ATmega328PB-A, U102 LMT84DCK

Commit message: Fixing
Parts:
- removed R? (x2): 2.2K, Resistor_SMD:R_0603_1608Metric_Pad0.98x0.95mm_HandSolder, symbol Device:R
- added R105, R106: 2.2K, Resistor_SMD:R_0603_1608Metric_Pad0.98x0.95mm_HandSolder, symbol Device:R
Connections:
- net +3V3: now also R105.1, R106.1
- net GND: no longer D102.1 (K), U101.21 (GND), U101.5 (GND)
- net INT_IMU: no longer U101.26 (PC3)
- net MISO1: no longer U101.23 (PC0)
- net PC4: no longer U101.27 (PC4)
- net PC5: no longer U101.28 (PC5)
- net RST: no longer U101.29 (~{RESET}/PC6)
- net SCK1: no longer U101.24 (PC1)
- net SCL: now also R106.2
- net SCLK: no longer U101.17 (PB5)
- net SDA: now also R105.2
- net T_OUT1: no longer U101.25 (PC2)
- new net: U101.21 (GND), U101.5 (GND)
